Commit message: Update my_robot.xacro

File: urdf/my_robot.xacro (robot description, xacro)
@@ -7,4 +7,5 @@
     <child link="chassis" />
   </joint>
+  <!-- central chassis (with casters included) link -->
   <link name="chassis">
     <pose>0 0 0.1 0 0 0</pose>
@@ -30,4 +31,5 @@
       </geometry>
     </visual>
+    <!-- back caster definition -->
     <collision name='back_caster_collision'>
       <origin xyz="-0.15 0 -0.05" rpy="0 0 0" />
@@ -42,4 +44,5 @@
       </geometry>
     </visual>
+    <!-- front caster definition -->
     <collision name='front_caster_collision'>
       <origin xyz="0.15 0 -0.05" rpy="0 0 0" />
@@ -55,3 +58,69 @@
     </visual>
   </link>
+  <!-- left revolute wheel definition -->
+  <link name="left_wheel">
+    <inertial>
+      <mass value="5.0" />
+      <origin xyz="0 0 0" rpy="0 1.5707 1.5707" />
+      <inertia
+        ixx="0.1" ixy="0" ixz="0"
+        iyy="0.1" iyz="0"
+        izz="0.1"
+      />
+    </inertial>
+    <collision name="left_wheel_collision">
+      <origin xyz="0 0 0" rpy="0 1.5707 1.5707" />
+      <geometry>
+        <cylinder radius="0.1" length="0.05" />
+      </geometry>
+    </collision>
+    <visual name="left_wheel_visual">
+      <origin xyz="0 0 0" rpy="0 1.5707 1.5707" />
+      <geometry>
+        <cylinder radius="0.1" length="0.05" />
+      </geometry>
+    </visual>
+  </link>
+  <!-- right revolute wheel definition -->
+  <link name="right_wheel">
+    <inertial>
+      <mass value="5.0" />
+      <origin xyz="0 0 0" rpy="0 1.5707 1.5707" />
+      <inertia
+        ixx="0.1" ixy="0" ixz="0"
+        iyy="0.1" iyz="0"
+        izz="0.1"
+      />
+    </inertial>
+    <collision name="right_wheel_collision">
+      <origin xyz="0 0 0" rpy="0 1.5707 1.5707" />
+      <geometry>
+        <cylinder radius="0.1" length="0.05" />
+      </geometry>
+    </collision>
+    <visual name="right_wheel_visual">
+      <origin xyz="0 0 0" rpy="0 1.5707 1.5707" />
+      <geometry>
+        <cylinder radius="0.1" length="0.05" />
+      </geometry>
+    </visual>
+  </link>
+  <!-- left wheel joint -->
+  <joint type="continuous" name="left_wheel_hinge">
+    <origin xyz="0 0.15 0" rpy="0 0 0" />
+    <child link="left_wheel" />
+    <parent link="chassis" />
+    <axis xyz="0 1 0" rpy="0 0 0" />
+    <limit effort="10000" velocity="1000" />
+    <dynamics damping="1.0" friction="1.0" />
+  </joint>
+  <!-- right wheel joint -->
+  <joint type="continuous" name="right_wheel_hinge">
+    <origin xyz="0 -0.15 0" rpy="0 0 0" />
+    <child link="right_wheel" />
+    <parent link="chassis" />
+    <axis xyz="0 1 0" rpy="0 0 0" />
+    <limit effort="10000" velocity="1000" />
+    <dynamics damping="1.0" friction="1.0" />
+  </joint>
 </robot>

Commit message: Update my_robot.xacro

File: urdf/my_robot.xacro (robot description, xacro)
@@ -1,5 +1,5 @@
 <?xml version='1.0'?>
 <robot name="my_robot" xmlns:xacro="http://www.ros.org/wiki/xacro">
-  <!-- DEF: robot has core footprint, rectangular chassis, left and right wheels, and left and right casters.    -->
+  <!-- DEF: robot has core footprint, rectangular chassis, left and right wheels, and front and back casters.    -->
   <!--       all six objects have appearances and are connected through joints, creating the entire robot frame. -->
   <link name="robot_footprint" />
@@ -22,5 +22,5 @@
     </inertial>
     <!-- main body appearance defintion -->
-    <collision name="collision">
+    <collision name="chassis_collision">
       <origin xyz="0 0 0" rpy="0 0 0" />
       <geometry>
@@ -127,3 +127,28 @@
     <dynamics damping="1.0" friction="1.0" />
   </joint>
+  <!-- camera sensor definition  -->
+  <link name="camera">
+    <box_inertia m="0.1" x="0.05" y="0.05" z="0.05" />
+    <inertial>
+      <mass value="0.1" />
+      <origin xyz="0 0 0" rpy="0 0 0" />
+      <inertia
+         ixx="1e-6" ixy="0" ixz="0"
+         iyy="1e-6" iyz="0"
+         izz="1e-6"
+      />
+    </inertial>
+    <collision name="camera_collision">
+      <origin xyz="0 0 0" rpy="0 0 0" />
+      <geometry>
+        <box size="0.05 0.05 0.05" />
+      </geometry>
+    </collision>
+    <visual name="camera_visual">
+      <origin xyz="0 0 0" rpy="0 0 0" />
+      <geometry>
+        <box size="0.05 0.05 0.05" />
+      </geometry>
+    </visual>
+  </link>
 </robot>

Commit message: Update my_robot.xacro

File: urdf/my_robot.xacro (robot description, xacro)
@@ -129,5 +129,7 @@
   <!-- camera sensor definition  -->
   <link name="camera">
-    <box_inertia m="0.1" x="0.05" y="0.05" z="0.05" />
+    <box_inertia m="0.1" x="0.05" y="0.05" z="0.05">
+      <origin xyz="0 0 0" rpy="0 0 0" />
+    </box_inertia>
     <inertial>
       <mass value="0.1" />
@@ -152,3 +154,10 @@
     </visual>
   </link>
+  <!-- camera joint definition -->
+  <joint type="fixed" name="camera_joint">
+    <origin xyz="0.2 0 0" rpy="0 0 0" />
+    <child link="camera" />
+    <parent link="chassis" />
+    <axis xyz="0 1 0" rpy="0 0 0" />
+  </joint>
 </robot>

Commit message: Update my_robot.xacro

File: urdf/my_robot.xacro (robot description, xacro)
@@ -129,7 +129,5 @@
   <!-- camera sensor definition  -->
   <link name="camera">
-    <box_inertia m="0.1" x="0.05" y="0.05" z="0.05">
-      <origin xyz="0 0 0" rpy="0 0 0" />
-    </box_inertia>
+    <box_inertia m="0.1" x="0.05" y="0.05" z="0.05" />
     <inertial>
       <mass value="0.1" />

Commit message: Update my_robot.xacro

File: urdf/my_robot.xacro (robot description, xacro)
@@ -159,3 +159,34 @@
     <axis xyz="0 1 0" rpy="0 0 0" />
   </joint>
+  <!-- lidar sensor definition -->
+  <link name="hokuyo">
+    <inertial>
+      <mass value="1e-5" />
+      <origin xyz="0 0 0" rpy="0 0 0" />
+      <inertia
+         ixx="1e-6" ixy="0" ixz="0"
+         iyy="1e-6" iyz="0"
+         izz="1e-6"
+      />
+    </inertial>
+    <collision name="hokuyo_collision">
+      <origin xyz="0 0 0" rpy="0 0 0" />
+      <geometry>
+        <box size="0.1 0.1 0.1" />
+      </geometry>
+    </collision>
+    <visual name="hokuyo_visual">
+      <origin xyz="0 0 0" rpy="0 0 0" />
+      <geometry>
+        <mesh filename="package://my_robot/meshes/hokuyo.dae" />
+      </geometry>
+    </visual>
+  </link>
+  <!-- lidar joint definition -->
+  <joint type="fixed" name="hokuyo_joint">
+    <origin xyz="0.15 0 0.1" rpy="0 0 0" />
+    <child link="hokuyo" />
+    <parent link="chassis" />
+    <axis xyz="0 1 0" rpy="0 0 0" />
+  </joint>
 </robot>
