Commit message: Update my_robot.xacro

File: my_robot/urdf/my_robot.xacro (robot description, xacro)
@@ -27,5 +27,5 @@
       <origin xyz="0 0 0" rpy="0 0 0" />
       <geometry>
-        <box size=".4 .2 .1" />
+        <box size=".48 .24 .12" />
       </geometry>
     </collision>
@@ -33,31 +33,32 @@
       <origin xyz="0 0 0" rpy="0 0 0" />
       <geometry>
-        <box size=".4 .2 .1" />
+        <box size=".48 .24 .12" />
       </geometry>
+      <material>Gazebo/SkyBlue</material>
     </visual>
     <!-- back caster appearance definition -->
     <collision name='back_caster_collision'>
-      <origin xyz="-0.15 0 -0.05" rpy="0 0 0" />
+      <origin xyz="-0.18 0 -0.06" rpy="0 0 0" />
       <geometry>
-        <sphere radius="0.0499" />
+        <sphere radius="0.0599" />
       </geometry>
     </collision>
     <visual name='back_caster_visual'>
-      <origin xyz="-0.15 0 -0.05" rpy="0 0 0" />
+      <origin xyz="-0.18 0 -0.06" rpy="0 0 0" />
       <geometry>
-        <sphere radius="0.05" />
+        <sphere radius="0.06" />
       </geometry>
     </visual>
     <!-- front caster appearance definition -->
     <collision name='front_caster_collision'>
-      <origin xyz="0.15 0 -0.05" rpy="0 0 0" />
+      <origin xyz="0.18 0 -0.06" rpy="0 0 0" />
       <geometry>
-        <sphere radius="0.0499" />
+        <sphere radius="0.0599" />
       </geometry>
     </collision>
     <visual name='front_caster_visual'>
-      <origin xyz="0.15 0 -0.05" rpy="0 0 0" />
+      <origin xyz="0.18 0 -0.06" rpy="0 0 0" />
       <geometry>
-        <sphere radius="0.05" />
+        <sphere radius="0.06" />
       </geometry>
     </visual>
@@ -77,5 +78,5 @@
       <origin xyz="0 0 0" rpy="0 1.5707 1.5707" />
       <geometry>
-        <cylinder radius="0.1" length="0.05" />
+        <cylinder radius="0.12" length="0.06" />
       </geometry>
     </collision>
@@ -83,5 +84,5 @@
       <origin xyz="0 0 0" rpy="0 1.5707 1.5707" />
       <geometry>
-        <cylinder radius="0.1" length="0.05" />
+        <cylinder radius="0.12" length="0.06" />
       </geometry>
     </visual>
@@ -101,5 +102,5 @@
       <origin xyz="0 0 0" rpy="0 1.5707 1.5707" />
       <geometry>
-        <cylinder radius="0.1" length="0.05" />
+        <cylinder radius="0.12" length="0.06" />
       </geometry>
     </collision>
@@ -107,5 +108,5 @@
       <origin xyz="0 0 0" rpy="0 1.5707 1.5707" />
       <geometry>
-        <cylinder radius="0.1" length="0.05" />
+        <cylinder radius="0.12" length="0.06" />
       </geometry>
     </visual>
@@ -113,5 +114,5 @@
   <!-- left wheel joint (connected to chassis) -->
   <joint type="continuous" name="left_wheel_hinge">
-    <origin xyz="0 0.15 0" rpy="0 0 0" />
+    <origin xyz="0 0.18 0" rpy="0 0 0" />
     <child link="left_wheel" />
     <parent link="chassis" />
@@ -122,5 +123,5 @@
   <!-- right wheel joint (connected to chassis) -->
   <joint type="continuous" name="right_wheel_hinge">
-    <origin xyz="0 -0.15 0" rpy="0 0 0" />
+    <origin xyz="0 -0.18 0" rpy="0 0 0" />
     <child link="right_wheel" />
     <parent link="chassis" />

Commit message: Update my_robot.xacro

File: my_robot/urdf/my_robot.xacro (robot description, xacro)
@@ -35,5 +35,5 @@
         <box size=".48 .24 .12" />
       </geometry>
-      <material>Gazebo/SkyBlue</material>
+      <material name="Gazebo/SkyBlue" />
     </visual>
     <!-- back caster appearance definition -->

Commit message: Update my_robot.xacro

File: my_robot/urdf/my_robot.xacro (robot description, xacro)
@@ -35,5 +35,5 @@
         <box size=".48 .24 .12" />
       </geometry>
-      <material name="Gazebo/SkyBlue" />
+      <material>Gazebo/SkyBlue</material>
     </visual>
     <!-- back caster appearance definition -->
@@ -64,4 +64,7 @@
     </visual>
   </link>
+  <gazebo reference="chassis">
+    <material>Gazebo/Blue</material>
+  </gazebo>
   <!-- left continuous wheel definition -->
   <link name="left_wheel">
@@ -88,4 +91,7 @@
     </visual>
   </link>
+  <gazebo reference="left_wheel">
+    <material>Gazebo/Black</material>
+  </gazebo>
   <!-- right continuous wheel definition -->
   <link name="right_wheel">
@@ -112,4 +118,7 @@
     </visual>
   </link>
+  <gazebo reference="right_wheel">
+    <material>Gazebo/Black</material>
+  </gazebo>
   <!-- left wheel joint (connected to chassis) -->
   <joint type="continuous" name="left_wheel_hinge">

Commit message: Update my_robot.xacro

File: my_robot/urdf/my_robot.xacro (robot description, xacro)
@@ -35,5 +35,4 @@
         <box size=".48 .24 .12" />
       </geometry>
-      <material>Gazebo/SkyBlue</material>
     </visual>
     <!-- back caster appearance definition -->

Commit message: Update my_robot.xacro

File: my_robot/urdf/my_robot.xacro (robot description, xacro)
@@ -64,5 +64,5 @@
   </link>
   <gazebo reference="chassis">
-    <material>Gazebo/Blue</material>
+    <material>Gazebo/SkyBlue</material>
   </gazebo>
   <!-- left continuous wheel definition -->

Commit message: Update my_robot.xacro

File: my_robot/urdf/my_robot.xacro (robot description, xacro)
@@ -163,4 +163,7 @@
     </visual>
   </link>
+  <gazebo reference="camera">
+    <material>Gazebo/Red</material>
+  </gazebo>
   <!-- camera joint definition -->
   <joint type="fixed" name="camera_joint">

Commit message: Update my_robot.xacro

File: my_robot/urdf/my_robot.xacro (robot description, xacro)
@@ -168,5 +168,5 @@
   <!-- camera joint definition -->
   <joint type="fixed" name="camera_joint">
-    <origin xyz="0.2 0 0" rpy="0 0 0" />
+    <origin xyz="0.24 0 0" rpy="0 0 0" />
     <child link="camera" />
     <parent link="chassis" />
@@ -199,5 +199,5 @@
   <!-- lidar joint definition -->
   <joint type="fixed" name="hokuyo_joint">
-    <origin xyz="0.15 0 0.1" rpy="0 0 0" />
+    <origin xyz="0.16 0 0.12" rpy="0 0 0" />
     <child link="hokuyo" />
     <parent link="chassis" />
